File: eagle/norns-shield.sch (EAGLE design)
At the start: 80 parts, among them J1 TRS-IN, J2 TRS-OUT, J3 ISP-ROW, Q1 ASFL-12.288mhz, SW1 PVA1, SW2 PVA1, SW3 PVA1, U1 CS4270, X1 RASPI_BOARD_B+#_E3

Commit message: Flip Tip and Ring on IO jacks.
Connections:
- removed net N$11: J1.T, R7.2
- removed net N$12: J1.R, R9.2
- new net N$7: J1.T, R9.2
- new net N$8: J1.R, R7.2
- net N$15: now also J2.R; no longer J2.T
- net N$16: now also J2.T; no longer J2.R
